File: schematics/fret_board/fret_board.kicad_sch (KiCad schematic)
At the start: 1 part, among them U1 Raspberry_Pi_Pico

Commit message: Added schematic and PCB design to fret_board
Parts:
- removed U1: Raspberry_Pi_Pico, ScottoKeebs_MCU:Raspberry_Pi_Pico, symbol ScottoKeebs:MCU_Raspberry_Pi_Pico
- added J1: Conn_01x06, Connector_PinHeader_2.00mm:PinHeader_1x06_P2.00mm_Vertical, symbol Connector_Generic:Conn_01x06
- added SW1: Green, ScottoKeebs_Choc:Choc_V1, symbol Switch:SW_SPST
- added SW2: Red, ScottoKeebs_Choc:Choc_V1, symbol Switch:SW_SPST
- added SW3: Yellow, ScottoKeebs_Choc:Choc_V1, symbol Switch:SW_SPST
- added SW4: Blue, ScottoKeebs_Choc:Choc_V1, symbol Switch:SW_SPST
- added SW5: Orange, ScottoKeebs_Choc:Choc_V1, symbol Switch:SW_SPST
Connections:
- new net: J1.1 (Pin_1), SW1.2 (B)
- new net: J1.2 (Pin_2), SW2.2 (B)
- new net: J1.3 (Pin_3), SW3.2 (B)
- new net: J1.4 (Pin_4), SW4.2 (B)
- new net: J1.5 (Pin_5), SW5.2 (B)
- new net GND: J1.6 (Pin_6), SW1.1 (A), SW2.1 (A), SW3.1 (A), SW4.1 (A), SW5.1 (A)

Commit message: Flip fret_board connector
Connections:
- net GND: now also J1.1 (Pin_1); no longer J1.6 (Pin_6)
- net at SW1.2 (B): now also J1.6 (Pin_6); no longer J1.1 (Pin_1)
- net at J1.2 (Pin_2): now also SW5.2 (B); no longer SW2.2 (B)
- net at J1.3 (Pin_3): now also SW4.2 (B); no longer SW3.2 (B)
- net at J1.4 (Pin_4): now also SW3.2 (B); no longer SW4.2 (B)
- net at J1.5 (Pin_5): now also SW2.2 (B); no longer SW5.2 (B)
Changed lines of the file:
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@@
 	(symbol
 		(lib_id "Connector_Generic:Conn_01x06")
-		(at 172.72 83.82 0)
+		(at 172.72 86.36 0)
+		(mirror x)
 		(unit 1)
 		(exclude_from_sim no)
@@
 		(on_board yes)
 		(dnp no)
-		(fields_autoplaced yes)
 		(property "Reference" "J1"
-			(at 175.26 83.8199 0)
+			(at 175.26 86.3601 0)
 			(effects
 				(font
@@
 		)
 		(property "Value" "Conn_01x06"
-			(at 175.26 86.3599 0)
+			(at 175.26 83.8201 0)
 			(effects
 				(font
@@
 		)
 		(property "Footprint" "Connector_PinHeader_2.00mm:PinHeader_1x06_P2.00mm_Vertical"
-			(at 172.72 83.82 0)
+			(at 172.72 86.36 0)
 			(effects
 				(font
@@
 		)
 		(property "Datasheet" "~"
-			(at 172.72 83.82 0)
+			(at 172.72 86.36 0)
 			(effects
 				(font
@@
 		)
 		(property "Description" "Generic connector, single row, 01x06, script generated (kicad-library-utils/schlib/autogen/connector/)"
-			(at 172.72 83.82 0)
+			(at 172.72 86.36 0)
 			(effects
 				(font

Commit message: Use sunken choc V1 footprint for fretboard
Parts:
- SW1, SW2, SW3, SW4, SW5: footprint ScottoKeebs_Choc:Choc_V1 -> custom_footprints:Choc_V1_sunken
Changed lines of the file:
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@@
 			)
 		)
-		(property "Footprint" "ScottoKeebs_Choc:Choc_V1"
+		(property "Footprint" "custom_footprints:Choc_V1_sunken"
 			(at 142.24 87.63 0)
 			(effects
@@
 			)
 		)
-		(property "Footprint" "ScottoKeebs_Choc:Choc_V1"
+		(property "Footprint" "custom_footprints:Choc_V1_sunken"
 			(at 142.24 114.3 0)
 			(effects
@@
 			)
 		)
-		(property "Footprint" "ScottoKeebs_Choc:Choc_V1"
+		(property "Footprint" "custom_footprints:Choc_V1_sunken"
 			(at 142.24 96.52 0)
 			(effects
@@
 			)
 		)
-		(property "Footprint" "ScottoKeebs_Choc:Choc_V1"
+		(property "Footprint" "custom_footprints:Choc_V1_sunken"
 			(at 142.24 105.41 0)
 			(effects
@@
 			)
 		)
-		(property "Footprint" "ScottoKeebs_Choc:Choc_V1"
+		(property "Footprint" "custom_footprints:Choc_V1_sunken"
 			(at 142.24 78.74 0)
 			(effects

Commit message: Update fret_board, motherboard and strum_bar schematics
Parts:
- removed J1: Conn_01x06, Connector_PinHeader_2.00mm:PinHeader_1x06_P2.00mm_Vertical, symbol Connector_Generic:Conn_01x06
- added J1: Conn_01x08, Connector_PinHeader_2.00mm:PinHeader_1x08_P2.00mm_Vertical, symbol Connector_Generic:Conn_01x08
Connections:
- net GND: now also J1.1 (Pin_1)
- net at SW5.2 (B): now also J1.6 (Pin_6)
- net at SW4.2 (B): now also J1.5 (Pin_5)
- net at SW3.2 (B): now also J1.4 (Pin_4)
- net at SW2.2 (B): now also J1.3 (Pin_3)
- net at SW1.2 (B): now also J1.2 (Pin_2)
- no-connect marks 0 -> 2
Other:
- moved on the sheet: SW1, SW2, SW4, SW5
Changed lines of the file:
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@@
 		(color 0 0 0 0)
 	)
+	(no_connect
+		(at 167.64 73.66)
+	)
+	(no_connect
+		(at 167.64 76.2)
+	)
 	(wire
 		(pts
@@
 			(width 0)
 			(type default)
-		)
-	)
-	(symbol
-		(lib_id "Connector_Generic:Conn_01x06")
-		(at 172.72 86.36 0)
-		(mirror x)
-		(unit 1)
-		(exclude_from_sim no)
-		(in_bom yes)
-		(on_board yes)
-		(dnp no)
-		(property "Reference" "J1"
-			(at 175.26 86.3601 0)
-			(effects
-				(font
-					(size 1.27 1.27)
-				)
-				(justify left)
-			)
-		)
-		(property "Value" "Conn_01x06"
-			(at 175.26 83.8201 0)
-			(effects
-				(font
-					(size 1.27 1.27)
-				)
-				(justify left)
-			)
-		)
-		(property "Footprint" "Connector_PinHeader_2.00mm:PinHeader_1x06_P2.00mm_Vertical"
-			(at 172.72 86.36 0)
-			(effects
-				(font
-					(size 1.27 1.27)
-				)
-				(hide yes)
-			)
-		)
-		(property "Datasheet" "~"
-			(at 172.72 86.36 0)
-			(effects
-				(font
-					(size 1.27 1.27)
-				)
-				(hide yes)
-			)
-		)
-		(property "Description" "Generic connector, single row, 01x06, script generated (kicad-library-utils/schlib/autogen/connector/)"
-			(at 172.72 86.36 0)
-			(effects
-				(font
-					(size 1.27 1.27)
-				)
-				(hide yes)
-			)
-		)
-		(pin "4"
-		)
-		(pin "5"
-		)
-		(pin "3"
-		)
-		(pin "1"
-		)
-		(pin "2"
-		)
-		(pin "6"
-		)
-		(instances
-			(project ""
-				(path "/9d371a9e-2977-429d-aa3c-ee2d51781e3b"
-					(reference "J1")
-					(unit 1)
-				)
-			)
 		)
 	)
 	(symbol
 		(lib_id "Switch:SW_SPST")
-		(at 142.24 87.63 0)
+		(at 142.24 105.41 0)
 		(unit 1)
 		(exclude_from_sim no)
@@
 		(fields_autoplaced yes)
 		(property "Reference" "SW2"
-			(at 142.24 81.28 0)
+			(at 142.24 99.06 0)
 			(effects
 				(font
@@
 		)
 		(property "Value" "Red"
-			(at 142.24 83.82 0)
+			(at 142.24 101.6 0)
 			(effects
 				(font
@@
 		)
 		(property "Footprint" "custom_footprints:Choc_V1_sunken"
-			(at 142.24 87.63 0)
+			(at 142.24 105.41 0)
 			(effects
 				(font
@@
 		)
 		(property "Datasheet" "~"
-			(at 142.24 87.63 0)
+			(at 142.24 105.41 0)
 			(effects
 				(font
@@
 		)
 		(property "Description" "Single Pole Single Throw (SPST) switch"
-			(at 142.24 87.63 0)
+			(at 142.24 105.41 0)
 			(effects
 				(font
@@
 	(symbol
 		(lib_id "Switch:SW_SPST")
-		(at 142.24 114.3 0)
+		(at 142.24 78.74 0)
 		(unit 1)
 		(exclude_from_sim no)
@@
 		(fields_autoplaced yes)
 		(property "Reference" "SW5"
-			(at 142.24 108.3282 0)
+			(at 142.24 72.7682 0)
 			(effects
 				(font
@@
 		)
 		(property "Value" "Orange"
-			(at 142.24 110.8682 0)
+			(at 142.24 75.3082 0)
 			(effects
 				(font
@@
 		)
 		(property "Footprint" "custom_footprints:Choc_V1_sunken"
-			(at 142.24 114.3 0)
+			(at 142.24 78.74 0)
 			(effects
 				(font
@@
 		)
 		(property "Datasheet" "~"
-			(at 142.24 114.3 0)
+			(at 142.24 78.74 0)
 			(effects
 				(font
@@
 		)
 		(property "Description" "Single Pole Single Throw (SPST) switch"
-			(at 142.24 114.3 0)
+			(at 142.24 78.74 0)
 			(effects
 				(font
@@
 				(path "/9d371a9e-2977-429d-aa3c-ee2d51781e3b"
 					(reference "SW3")
+					(unit 1)
+				)
+			)
+		)
+	)
+	(symbol
+		(lib_id "Connector_Generic:Conn_01x08")
+		(at 172.72 83.82 0)
+		(mirror x)
+		(unit 1)
+		(exclude_from_sim no)
+		(in_bom yes)
+		(on_board yes)
+		(dnp no)
+		(property "Reference" "J1"
+			(at 175.26 83.8201 0)
+			(effects
+				(font
+					(size 1.27 1.27)
+				)
+				(justify left)
+			)
+		)
+		(property "Value" "Conn_01x08"
+			(at 175.26 81.2801 0)
+			(effects
+				(font
+					(size 1.27 1.27)
+				)
+				(justify left)
+			)
+		)
+		(property "Footprint" "Connector_PinHeader_2.00mm:PinHeader_1x08_P2.00mm_Vertical"
+			(at 172.72 83.82 0)
+			(effects
+				(font
+					(size 1.27 1.27)
+				)
+				(hide yes)
+			)
+		)
+		(property "Datasheet" "~"
+			(at 172.72 83.82 0)
+			(effects
+				(font
+					(size 1.27 1.27)
+				)
+				(hide yes)
+			)
+		)
+		(property "Description" "Generic connector, single row, 01x08, script generated (kicad-library-utils/schlib/autogen/connector/)"
+			(at 172.72 83.82 0)
+			(effects
+				(font
+					(size 1.27 1.27)
+				)
+				(hide yes)
+			)
+		)
+		(pin "6"
+		)
+		(pin "2"
+		)
+		(pin "5"
+		)
+		(pin "4"
+		)
+		(pin "3"
+		)
+		(pin "1"
+		)
+		(pin "8"
+		)
+		(pin "7"
+		)
+		(instances
+			(project ""
+				(path "/9d371a9e-2977-429d-aa3c-ee2d51781e3b"
+					(reference "J1")
 					(unit 1)
 				)
@@
 	(symbol
 		(lib_id "Switch:SW_SPST")
-		(at 142.24 105.41 0)
+		(at 142.24 87.63 0)
 		(unit 1)
 		(exclude_from_sim no)
@@
 		(fields_autoplaced yes)
 		(property "Reference" "SW4"
-			(at 142.24 99.4382 0)
+			(at 142.24 81.6582 0)
 			(effects
 				(font
@@
 		)
 		(property "Value" "Blue"
-			(at 142.24 101.9782 0)
+			(at 142.24 84.1982 0)
 			(effects
 				(font
@@
 		)
 		(property "Footprint" "custom_footprints:Choc_V1_sunken"
-			(at 142.24 105.41 0)
+			(at 142.24 87.63 0)
 			(effects
 				(font
@@
 		)
 		(property "Datasheet" "~"
-			(at 142.24 105.41 0)
+			(at 142.24 87.63 0)
 			(effects
 				(font
@@
 		)
 		(property "Description" "Single Pole Single Throw (SPST) switch"
-			(at 142.24 105.41 0)
+			(at 142.24 87.63 0)
 			(effects
 				(font
@@
 	(symbol
 		(lib_id "Switch:SW_SPST")
-		(at 142.24 78.74 0)
+		(at 142.24 114.3 0)
 		(unit 1)
 		(exclude_from_sim no)
@@
 		(on_board yes)
 		(dnp no)
-		(fields_autoplaced yes)
 		(property "Reference" "SW1"
-			(at 142.24 72.39 0)
+			(at 142.24 107.95 0)
 			(effects
 				(font
@@
 		)
 		(property "Value" "Green"
-			(at 142.24 74.93 0)
+			(at 142.24 110.49 0)
 			(effects
 				(font
@@
 		)
 		(property "Footprint" "custom_footprints:Choc_V1_sunken"
-			(at 142.24 78.74 0)
+			(at 142.24 114.3 0)
 			(effects
 				(font
@@
 		)
 		(property "Datasheet" "~"
-			(at 142.24 78.74 0)
+			(at 142.24 114.3 0)
 			(effects
 				(font
@@
 		)
 		(property "Description" "Single Pole Single Throw (SPST) switch"
-			(at 142.24 78.74 0)
-			(effects
-				(font
+			(at 142.24 114.3 0)
+			(effects
+				(font
