File: schematics/strum_bar/strum_bar.kicad_pcb (KiCad board)
At the start: 2 copper layers, 56 x 57.3 mm, 3 parts, among them J1 Conn_01x03, SW1 STRUM_UP, SW2 STRUM_DOWN

Commit message: Add silkscreen graphics to each schematic
Parts:
- added G***: LOGO, LOGO, B.Cu at (135.6, 89.7)
